Commit message: Sync with latest autoware

File: sample_vehicle_description/urdf/vehicle.xacro (robot description, xacro)
@@ -6,7 +6,7 @@
   <link name="base_link">
     <visual>
-      <origin xyz="${vehicle_info['/**']['ros__parameters']['wheel_base']/2.0} 0 0" rpy="${pi/2.0} 0 ${pi}"/>
+      <origin xyz="0 0 0" rpy="0 0 ${pi/2}"/>
       <geometry>
-        <mesh filename="package://sample_vehicle_description/mesh/lexus.dae" scale="1 1 1"/>
+        <mesh filename="package://sample_vehicle_description/mesh/buggy_rviz.dae" scale="1 1 1"/>
       </geometry>
     </visual>

Commit message: added tars5 model

File: sample_vehicle_description/urdf/vehicle.xacro (robot description, xacro)
@@ -6,7 +6,7 @@
   <link name="base_link">
     <visual>
-      <origin xyz="0 0 0" rpy="0 0 ${pi/2}"/>
+      <origin xyz="0 0 0" rpy="0 0 0"/>
       <geometry>
-        <mesh filename="package://sample_vehicle_description/mesh/buggy_rviz.dae" scale="1 1 1"/>
+        <mesh filename="package://sample_vehicle_description/mesh/base_link.STL" scale="1 1 1"/>
       </geometry>
     </visual>
